File: GPSReceiver_Kenwood710_tiny.brd (EAGLE design)
At the start: 35 x 50 mm, 13 parts, among them U1 MAX232PTH

Commit message: more clearence
more clearence
Parts:
- moved JP2 2.16 mm to (32.7, 3.70)
- moved C1 1.00 mm to (37.8, 43.0)
- moved C2 1.00 mm to (38.0, 36.5)
- moved C3 1.00 mm to (30.0, 43.0)
- moved C4 1.00 mm to (38.0, 30.0)
- moved C5 1.00 mm to (30.0, 36.5)
- moved C6 1.00 mm to (30.0, 30.0)
- moved JP1 1.00 mm to (56.5, 44.5)
- moved JP3 1.00 mm to (56.5, 35.0)
- moved U1 1.00 mm to (48.5, 36.5)
Routing:
- net N$5: track 31.0 -> 27.5 mm
- net 5V: track 64.7 -> 67.9 mm
- net VIN: track 22.5 -> 19.9 mm
- net TX_UB: track 31.2 -> 33.4 mm
